File: pcb/ESPHome-Indoor-Multi-Sensor.kicad_pcb (KiCad board)
At the start: 4 copper layers, 52.5 x 59.7 mm, 106 parts, among them J1 SEN66, J2 USB-C, J3 SEN0609, J4 LD2410, J5 SPKR, J6 LD2450, Q1 MMBFJ201, SW1 BOOT, SW2 RESET, U1 TPS22917DBV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

Commit message: Minor changes
Separate SEN66 on a separate I2C bus.
Add WIFi Antenna cutout.
Beef-up Power and Ground connections to SEN66.
Parts:
- added R22: 5.1KΩ, Resistor_SMD:R_0402_1005Metric, F.Cu at (136.2, 79.9)
- added R23: 5.1KΩ, Resistor_SMD:R_0402_1005Metric, F.Cu at (135.2, 79.9)
- R8, R9: value DNP -> 5.1KΩ
Connections:
- J1 pad 3: /SDA -> /SDA2
- J1 pad 4: /SCL -> /SCL2
- R8 pad 2: /SDA -> /SDA1
- R9 pad 2: /SCL -> /SCL1
- U10 pad 1: /SCL -> /SCL1
- U10 pad 6: /SDA -> /SDA1
- U11 pad 3: /SDA -> /SDA1
- U11 pad 6: /SCL -> /SCL1
- U12 pad 10: /SDA -> /SDA1
- U12 pad 9: /SCL -> /SCL1
- U13 pad 2: /SCL -> /SCL1
- U13 pad 4: /SDA -> /SDA1
- U15 pad 10: /SCL -> /SCL1
- U15 pad 9: /SDA -> /SDA1
- U16 pad 1: /SDA -> /SDA1
- U16 pad 2: /SCL -> /SCL1
- U8 pad 24: /SCL -> /SCL1
- U8 pad 25: /SDA -> /SDA1
- U8 pad 36: unconnected-(U8-RXD0-Pad36) -> /SCL2
- U8 pad 37: unconnected-(U8-TXD0-Pad37) -> /SDA2
- U9 pad 4: /SDA -> /SDA1
- U9 pad 5: /SCL -> /SCL1
Routing:
- net /SDA: track 122.7 -> 0.00 mm, vias 8 -> 0
- net /SDA1: track 0.00 -> 121.0 mm, vias 0 -> 8
- net /SCL: track 120.9 -> 0.00 mm, vias 9 -> 0
- net /SCL1: track 0.00 -> 115.1 mm, vias 0 -> 7
- net /Presence Sensors/LD24X0_VCC: track 56.0 -> 19.3 mm
- net GND: track 190.1 -> 163.1 mm, vias 76 -> 75
- net /SCL2: track 0.00 -> 26.6 mm, vias 0 -> 2
- net /SDA2: track 0.00 -> 26.1 mm, vias 0 -> 2
- net +3.3VA: track 108.4 -> 113.0 mm
- added copper zone on In2.Cu, net /Presence Sensors/LD24X0_VCC
Other:
- outline, holes or cut-outs redrawn
- board text added: "REV A 04-10-2025"
- board text removed: "REV - 04-10-2025"
