File: pcb/Env-Sensors-1.kicad_sch (KiCad schematic)
At the start: 13 parts, among them J1 SEN66, U11 SGP41, U12 SCD41, U16 SHT45

Commit message: Minor changes
Separate SEN66 on a separate I2C bus.
Add WIFi Antenna cutout.
Beef-up Power and Ground connections to SEN66.
Parts:
- added R22, R23: 5.1KΩ, Resistor_SMD:R_0402_1005Metric, symbol Device:R
Connections:
- net +3.3VA: now also R22.1, R23.1
- net SCL renamed SCL1
- net SCL1: no longer J1.4 (Pin_4)
- net SDA renamed SDA1
- net SDA1: no longer J1.3 (Pin_3)
- new net SCL2: J1.4 (Pin_4), R22.2
- new net SDA2: J1.3 (Pin_3), R23.2
Other:
- note added: "Bath or Kitchen Set"
- note added: "I^{2}C2 Pullup"
- note added: "Notes 1. Recommend one of two configurations. A. SEN66. B. SHT45, SCD41 and SGP41 for Bath or Kitchen. 2. Temperature & Humidity Sensor can be SHT40 , SHT41, or SHT45 for increasing accuracy. 3. CO^{2} (SCD40 or SCD41) measures CO^{2}, Temperature and Humidity. 4. Air Quality Sensor (SGP40 or SGP41) measures VOC, NO_{X}. These sensors are self heating and not recommended for measuring room temper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"
- note removed: "Discrete Sensor Set"
- note removed: "Notes 1. Recommend one of two configurations. A. SEN66. B. SHT45, SCD41 and SGP41. 2. Temperature & Humidity Sensor can be SHT40 , SHT41, or SHT45 for increasing accuracy. 3. CO^{2} (SCD40 or SCD41) measures CO^{2}, Temperature and Humidity. 4. Air Quality Sensor (SGP40 or SGP41) measures VOC, NO_{X}. These sensors are self heating and not recommended for measuring room temperature. 5. SEN66 meas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"
